File: pcb/atomic_36.kicad_pcb (KiCad board)
At the start: 2 copper layers, 133.9 x 99 mm, 47 parts, among them J1 USB_C_12P

Commit message: Add ground plane and silkscreen labels
Routing:
- net GND: track 86.2 -> 11.9 mm, vias 0 -> 7
- net GP8: track 64.5 -> 66.8 mm
- net GP9: track 66.8 -> 68.0 mm
- added copper zone on B.Cu, net GND
- added copper zone on F.Cu, net GND
Other:
- board text added: "3V3"
- board text added: "5V"
- board text added: "GND"
- board text added: "P0"
- board text added: "P1"
- board text added: "P10"
- board text added: "P11"
- board text added: "P12"
- board text added: "P13"
- board text added: "P14"
- board text added: "P15"
- board text added: "P2"
- board text added: "P26"
- board text added: "P27"
- board text added: "P28"
- board text added: "P29"
- board text added: "P3"
- board text added: "P4"
- board text added: "P5"
- board text added: "P6"
- board text added: "P7"
- board text added: "P8"
- board text added: "P9"
- board text added: "USBC"
- board text added: "atomic"

Commit message: Add final tweaks to PCB before ordering
Routing:
- net P5V: track 133.1 -> 132.2 mm
Other:
- board text added: "v0.1.0"
